File: Project2_WeevilEyeMod/WeevilEyeMod.kicad_pcb (KiCad board)
At the start: 2 copper layers, 0 parts

Commit message: Updating plan for Session 3
Parts:
- added BT1: Battery_Cell, Battery:BatteryHolder_ComfortableElectronic_CH273-2450_1x2450, B.Cu at (73.5, 98.5)
- added D1: LED, LED_THT:LED_D5.0mm, F.Cu at (103.3, 89.8)
- added D2: LED, LED_THT:LED_D5.0mm, F.Cu at (95.0, 79.6)
- added Q1: 2N3904, Package_TO_SOT_THT:TO-92_Inline_Wide, F.Cu at (85.0, 71.1)
- added R1: 47K, Resistor_THT:R_Axial_DIN0204_L3.6mm_D1.6mm_P7.62mm_Horizontal, F.Cu at (104.9, 99.2)
- added R2: 220R, Resistor_THT:R_Axial_DIN0204_L3.6mm_D1.6mm_P7.62mm_Horizontal, F.Cu at (101.0, 77.4)
- added R3: LDR07, OptoDevice:R_LDR_5.1x4.3mm_P3.4mm_Vertical, F.Cu at (75.8, 75.8)
- added R4: 220R, Resistor_THT:R_Axial_DIN0204_L3.6mm_D1.6mm_P7.62mm_Horizontal, F.Cu at (107.0, 81.7)
Routing:
- net Net-(BT1-+): track 0.00 -> 68.3 mm, vias 0 -> 1
- net Net-(Q1-B): track 0.00 -> 58.2 mm, vias 0 -> 1
- net GND: track 0.00 -> 43.8 mm
- net Net-(Q1-C): track 0.00 -> 19.3 mm
- net Net-(D1-K): track 0.00 -> 13.4 mm, vias 0 -> 1
- net Net-(D2-K): track 0.00 -> 12.9 mm
Other:
- board outline added: 54 x 54 mm
